File: Aaram.kicad_sch (KiCad schematic)
At the start: 73 parts, among them J1 Conn_01x03, J10 Conn_01x03_Socket, J11 Conn_01x03_Socket, J12 Conn_01x03_Socket, J13 Conn_01x03_Socket, J2 Conn_01x02, J3 AC_OUT, J4 SWITCH_IN, J5 PSU_5V_OUT, J6 PSU_AC_IN, J7 Conn_01x05, J8 USB_C_Receptacle_USB2.0_16P, J9 Conn_01x02, K1 10A cube relay, K2 10A cube relay, K3 10A cube relay, Q1 BT136-600, Q2 2N2222A, Q3 2N2222A, Q4 2N2222A, SW1 SW_Push, SW2 SW_Push, SW4 SW_Push, U1 ESP32-C6-MINI-1/U, U2 AZ1117D-3.3TRE1, U5 TLP281-4GB_F_

Commit message: Big Update
Parts:
- removed C2: 10uf, PCM_Capacitor_SMD_Handsoldering_AKL:C_1206_3216Metric_Pad1.42x1.75mm, symbol PCM_Capacitor_AKL:CP_Radial_D10.0mm_P5.00mm
- removed J7: Conn_01x05, Connector_PinHeader_2.54mm:PinHeader_1x05_P2.54mm_Vertical, symbol Connector_Generic:Conn_01x05
- added J10, J11: Conn_01x03, Connector_PinSocket_2.54mm:PinSocket_1x03_P2.54mm_Vertical, symbol Connector_Generic:Conn_01x03
- added Q5: BC817-25, Package_TO_SOT_SMD:TSOT-23_HandSoldering, symbol PCM_Transistor_BJT_AKL:2N2222A
- added R11: 30, PCM_Resistor_SMD_AKL:R_1206_3216Metric_Pad1.42x1.75mm_HandSolder, symbol PCM_Resistor_AKL:R_1206
- added R13: 50, PCM_Resistor_SMD_AKL:R_1206_3216Metric_Pad1.42x1.75mm_HandSolder, symbol PCM_Resistor_AKL:R_1206
- added R16: 10k, PCM_Resistor_SMD_AKL:R_1206_3216Metric_Pad1.42x1.75mm_HandSolder, symbol PCM_Resistor_AKL:R_1206
- D1, D2, D3: value 1N4007 -> 1N5819WT
- Q2, Q3, Q4: value 2N2222A -> BC817-25; footprint PCM_Package_TO_SOT_THT_AKL:TO-18-3_EBC -> Package_TO_SOT_SMD:TSOT-23_HandSoldering
- R15, R17, R19, R23, R5, R7: footprint PCM_Resistor_SMD_AKL:R_1206_3216Metric_Pad1.42x1.75mm_HandSolder -> PCM_Resistor_SMD_AKL:R_2512_6332Metric_Pad1.52x3.35mm_HandSolder
- R6: value 330 -> 390; footprint PCM_Resistor_SMD_AKL:R_1206_3216Metric_Pad1.42x1.75mm_HandSolder -> PCM_Resistor_SMD_AKL:R_2512_6332Metric_Pad1.52x3.35mm_HandSolder
- R8: value 100K -> 2k
- R9: value 100K -> 1k
- renumbered J11 to Switch_1, J12 to Switch_2, J13 to Switch_3, J10 to Switch_4
Connections:
- net SP1 is gone; now on net Sensor 1: U1.13 (GPIO1/ADC1_CH1/XTAL_32K_N)
- net SP3 is gone; now on net D1: U1.6 (GPIO3/ADC1_CH3)
- net +3.3V: now also Q5.3 (C)
- net +5V: now also J10.3 (Pin_3), R16.1; no longer R9.1
- net AC_IN_1: now also R26.2, Switch_1.2 (Pin_2), U1.27 (GPIO21); no longer D8.3 (1), J4.1 (Pin_1), R27.2, Switch_4.2 (Pin_2), U1.19 (GPIO14)
- net AC_IN_2: now also R25.2, Switch_2.2 (Pin_2), U1.26 (GPIO20); no longer D9.3 (1), J4.2 (Pin_2), R26.2, Switch_1.2 (Pin_2), U1.20 (GPIO15)
- net AC_IN_3: now also R20.2, Switch_3.2 (Pin_2), U1.29 (GPIO23); no longer D10.3 (1), J4.3 (Pin_3), R25.2, Switch_2.2 (Pin_2), U1.24 (GPIO18)
- net AC_IN_4: now also R27.2, Switch_4.2 (Pin_2), U1.28 (GPIO22); no longer D11.3 (1), J4.4 (Pin_4), R20.2, Switch_3.2 (Pin_2), U1.25 (GPIO19)
- net AC_L: no longer J6.1 (Pin_1)
- net D1: no longer U1.28 (GPIO22)
- net D2: now also U1.19 (GPIO14); no longer U1.27 (GPIO21)
- net D3: now also U1.24 (GPIO18); no longer U1.26 (GPIO20)
- net GND: now also J2.1 (Pin_1), J10.2 (Pin_2), J11.1 (Pin_1)
- net LOAD_1: now also J3.4 (Pin_4), RV2.1; no longer J3.3 (Pin_3), RV3.1
- net LOAD_2: now also J3.3 (Pin_3), RV3.1; no longer J3.2 (Pin_2), RV2.1
- net LOAD_3: now also J3.2 (Pin_2); no longer J3.4 (Pin_4)
- net Sensor 1: no longer U1.15 (MTCK/GPIO6/ADC1_CH6)
- net T1_Pin: now also U1.25 (GPIO19); no longer U1.29 (GPIO23)
- net at C19.2, R21.1, SW4.2: now also U1.23 (GPIO9); no longer U1.22 (GPIO8)
- net AC_L_MAIN: now reaches F1.2, J3.6 (Pin_6)
- net AC_L_MAIN: now also J6.1 (Pin_1)
- net IR_IN: now reaches R8.1, R9.2
- net IR_IN: now also U1.12 (GPIO0/ADC1_CH0/XTAL_32K_P); no longer J2.1 (Pin_1)
- net at J9.1 (Pin_1): now also U4.6 (B_IN-); no longer U4.5 (B_IN+)
- net at J9.2 (Pin_2): now also U4.5 (B_IN+); no longer U4.6 (B_IN-)
- net at R22.2: now also U1.22 (GPIO8); no longer U1.23 (GPIO9)
- net at U1.30 (U0RXD/GPIO17): now also J11.3 (Pin_3)
- net at U1.31 (U0TXD/GPIO16): now also J11.2 (Pin_2)
- net G1: no longer names the net of D8.2 (-), U5.2 (C1)
- net G2: no longer names the net of D9.2 (-), U5.4 (C2)
- net G3: no longer names the net of D10.2 (-), U5.6 (C3)
- net G4: no longer names the net of D11.2 (-), U5.8 (C4)
- net SP2 renamed IR_OUT
- net IR_OUT: now also R13.2
- net SP4: no longer names the net of U1.9 (MTMS/GPIO4/ADC1_CH4)
- net SP5: no longer names the net of U1.10 (MTDI/GPIO5/ADC1_CH5)
- net Sensor 2: no longer names the net of J2.2 (Pin_2)
- net Sensor 2: now also R11.1; no longer U1.16 (MTDO/GPIO7)
- net USB+: no longer names the net of J8.A6 (D+), J8.B6 (D+), U1.18 (GPIO13/USB_D+)
- net USB-: no longer names the net of J8.A7 (D-), J8.B7 (D-), U1.17 (GPIO12/USB_D-)
- new net: Q5.1 (E), R11.2
- new net: Q5.2 (B), R13.1
- new net: J10.1 (Pin_1), R16.2, R9.1
- new net S1: D8.3 (1), J4.1 (Pin_1)
- new net S2: D9.3 (1), J4.2 (Pin_2)
- new net S3: D10.3 (1), J4.3 (Pin_3)
- new net S4: D11.3 (1), J4.4 (Pin_4)
- no-connect marks 6 -> 10
Other:
- note added: "10uf"
- note added: "AARAM"
- note added: "Debug"
- note added: "ESP32_C6"
- note added: "IR Receiver"
- note added: "IR Transmitter"
- note added: "Physical switch input by using either rectified AC signal from the Opto or the TTP223 module."
- note added: "Pins"
- note added: "Relay and Triac"
- note added: "Rocker Switches -> Rectifier Opto -> ESP the switches already have live connected"
- note added: "SX are old rocker switches in the switch board. AC_N is neutral"
- note added: "Sensor input"
- note added: "Stuff"
- note added: "TP4056 and Mini Boost converter"
- note added: "These are the connections for female header"
- note added: "V G D"
- note removed: "ESP32_C6_MINI"
- note removed: "I'm taking the output from the switch board switches that already have Live connected and rectifying them for the TLP281 opto to give a digital signal the ESP"
- note removed: "Relay_1"
- note removed: "Relay_2"
- note removed: "Relay_3"
- note removed: "SENSORS"
- note removed: "SP are spare pins"
- note removed: "Spare ESP pins"
- note removed: "Triac_1"
- note removed: "USB"
- note removed: "VRM"
- note removed: "ZMCT103C"
- title: (none) -> Aaram - Home Automation
- moved on the sheet: C11, C12, C16, C6, C7, D2, D3, K1, K2, K3, RV1, RV2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
