File: Aaram.kicad_pcb (KiCad board)
At the start: 2 copper layers, 100 x 100 mm, 73 parts, among them J1 Conn_01x03, J10 Conn_01x03_Socket, J11 Conn_01x03_Socket, J12 Conn_01x03_Socket, J13 Conn_01x03_Socket, J2 Conn_01x02, J3 AC_OUT, J4 SWITCH_IN, J5 PSU_5V_OUT, J6 PSU_AC_IN, J7 Conn_01x05, J8 USB_C_Receptacle_USB2.0_16P, J9 Conn_01x02, K1 10A cube relay, K2 10A cube relay, K3 10A cube relay, Q1 BT136-600, Q2 2N2222A, Q3 2N2222A, Q4 2N2222A, SW1 SW_Push, SW2 SW_Push, SW4 SW_Push, U1 ESP32-C6-MINI-1/U, U2 AZ1117D-3.3TRE1, U5 TLP281-4GB_F_

Commit message: Big Update
Parts:
- removed C2: 10uf, PCM_Capacitor_SMD_Handsoldering_AKL:C_1206_3216Metric_Pad1.42x1.75mm
- removed J12, J13: Conn_01x03_Socket, Connector_JST:JST_SH_BM03B-SRSS-TB_1x03-1MP_P1.00mm_Vertical
- removed J7: Conn_01x05, Connector_PinHeader_2.54mm:PinHeader_1x05_P2.54mm_Vertical
- added Q5: BC817-25, Package_TO_SOT_SMD:TSOT-23_HandSoldering, F.Cu at (83.6, 32.5)
- added R11: 30, PCM_Resistor_SMD_AKL:R_1206_3216Metric_Pad1.42x1.75mm_HandSolder, F.Cu at (83.2, 29.0)
- added R13: 50, PCM_Resistor_SMD_AKL:R_1206_3216Metric_Pad1.42x1.75mm_HandSolder, F.Cu at (87.6, 27.6)
- added R16: 10k, PCM_Resistor_SMD_AKL:R_1206_3216Metric_Pad1.42x1.75mm_HandSolder, F.Cu at (78.9, 33.3)
- added Switch_1: Conn_01x03_Socket, Connector_JST:JST_SH_BM03B-SRSS-TB_1x03-1MP_P1.00mm_Vertical, B.Cu at (101.0, 59.5)
- added Switch_2: Conn_01x03_Socket, Connector_JST:JST_SH_BM03B-SRSS-TB_1x03-1MP_P1.00mm_Vertical, B.Cu at (101.0, 50.2)
- added Switch_3: Conn_01x03_Socket, Connector_JST:JST_SH_BM03B-SRSS-TB_1x03-1MP_P1.00mm_Vertical, B.Cu at (113.9, 50.2)
- added Switch_4: Conn_01x03_Socket, Connector_JST:JST_SH_BM03B-SRSS-TB_1x03-1MP_P1.00mm_Vertical, B.Cu at (113.9, 59.5)
- C1, C4, F1, J1, J2, J3, J4, J5, J6, J9, K1, K2, K3, OC1, Q1, RV1, RV2, RV3, RV4, SW1, SW2, SW4: moved to B.Cu
- D1, D2, D3: value 1N4007 -> 1N5819WT; moved to F.Cu
- J10, J11: value Conn_01x03_Socket -> Conn_01x03; footprint Connector_JST:JST_SH_BM03B-SRSS-TB_1x03-1MP_P1.00mm_Vertical -> Connector_PinSocket_2.54mm:PinSocket_1x03_P2.54mm_Vertical; moved to B.Cu
- Q2, Q3, Q4: value 2N2222A -> BC817-25; footprint PCM_Package_TO_SOT_THT_AKL:TO-18-3_EBC -> Package_TO_SOT_SMD:TSOT-23_HandSoldering
- R15, R17, R19, R23, R5, R7: footprint PCM_Resistor_SMD_AKL:R_1206_3216Metric_Pad1.42x1.75mm_HandSolder -> PCM_Resistor_SMD_AKL:R_2512_6332Metric_Pad1.52x3.35mm_HandSolder
- R20, R25, R26, R27: moved to F.Cu
- R6: value 330 -> 390; footprint PCM_Resistor_SMD_AKL:R_1206_3216Metric_Pad1.42x1.75mm_HandSolder -> PCM_Resistor_SMD_AKL:R_2512_6332Metric_Pad1.52x3.35mm_HandSolder
- R8: value 100K -> 2k
- R9: value 100K -> 1k
- moved D3 75.3 mm to (30.4, 60.9), turned to 0 degrees
- moved K2 70.5 mm to (30.4, 67.0), turned to -90 degrees
- moved J3 62.3 mm to (82.3, 109.3), turned to 180 degrees
- moved RV4 58.4 mm to (90.3, 109.3), turned to -45 degrees
- moved J10 49.3 mm to (78.9, 28.4), turned to 0 degrees
- moved C1 39.0 mm to (79.7, 73.8), turned to -90 degrees
- moved C7 37.6 mm to (59.6, 24.3), turned to 90 degrees
- moved C12 36.9 mm to (72.5, 24.3), turned to -90 degrees
- moved Q1 35.3 mm to (81.7, 95.0), turned to 90 degrees
- moved D1 34.9 mm to (67.7, 60.9), turned to 0 degrees
- moved C11 34.5 mm to (75.7, 24.3), turned to -90 degrees
- moved RV2 34.5 mm to (36.5, 87.9), turned to -70 degrees
- moved J11 34.3 mm to (109.0, 27.1), turned to 180 degrees
- moved RV1 34.0 mm to (71.2, 87.9), turned to -70 degrees
- moved C6 33.7 mm to (56.3, 24.3), turned to 90 degrees
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Connections:
- net G1 renamed Net-(D8--)
- net G2 renamed Net-(D9--)
- net G3 renamed Net-(D10--)
- net G4 renamed Net-(D11--)
- net USB+ renamed Net-(U1-GPIO13/USB_D+)
- net USB- renamed Net-(U1-GPIO12/USB_D-)
- C19 pad 2: Net-(U1-GPIO8) -> Net-(U1-GPIO9)
- D10 pad 3: AC_IN_3 -> S3
- D11 pad 3: AC_IN_4 -> S4
- D8 pad 3: AC_IN_1 -> S1
- D9 pad 3: AC_IN_2 -> S2
- F1 pad 2: Net-(J3-Pin_6) -> AC_L_MAIN
- J10 pad 1: +3.3V -> Net-(J10-Pin_1)
- J10 pad 2: AC_IN_1 -> GND
- J10 pad 3: GND -> +5V
- J11 pad 1: +3.3V -> GND
- J11 pad 2: AC_IN_2 -> Net-(J11-Pin_2)
- J11 pad 3: GND -> Net-(J11-Pin_3)
- J2 pad 1: Net-(J2-Pin_1) -> GND
- J2 pad 2: Sensor 2 -> Net-(J2-Pin_2)
- J3 pad 2: LOAD_2 -> LOAD_3
- J3 pad 3: LOAD_1 -> LOAD_2
- J3 pad 4: LOAD_3 -> LOAD_1
- J3 pad 6: Net-(J3-Pin_6) -> AC_L_MAIN
- J4 pad 1: AC_IN_1 -> S1
- J4 pad 2: AC_IN_2 -> S2
- J4 pad 3: AC_IN_3 -> S3
- J4 pad 4: AC_IN_4 -> S4
- J6 pad 1: AC_L -> AC_L_MAIN
- R20 pad 2: AC_IN_4 -> AC_IN_3
- R21 pad 1: Net-(U1-GPIO8) -> Net-(U1-GPIO9)
- R22 pad 2: Net-(U1-GPIO9) -> Net-(U1-GPIO8)
- R25 pad 2: AC_IN_3 -> AC_IN_2
- R26 pad 2: AC_IN_2 -> AC_IN_1
- R27 pad 2: AC_IN_1 -> AC_IN_4
- R8 pad 1: Net-(J2-Pin_1) -> IR_IN
- R9 pad 1: +5V -> Net-(J10-Pin_1)
- R9 pad 2: Net-(J2-Pin_1) -> IR_IN
- RV2 pad 1: LOAD_2 -> LOAD_1
- RV3 pad 1: LOAD_1 -> LOAD_2
- SW4 pad 2: Net-(U1-GPIO8) -> Net-(U1-GPIO9)
- U1 pad 10: SP5 -> unconnected-(U1-MTDI/GPIO5/ADC1_CH5-Pad10)
- U1 pad 12: unconnected-(U1-GPIO0/ADC1_CH0/XTAL_32K_P-Pad12) -> IR_IN
- U1 pad 13: SP1 -> Sensor 1
- U1 pad 15: Sensor 1 -> unconnected-(U1-MTCK/GPIO6/ADC1_CH6-Pad15)
- U1 pad 16: Sensor 2 -> unconnected-(U1-MTDO/GPIO7-Pad16)
- U1 pad 19: AC_IN_1 -> D2
- U1 pad 20: AC_IN_2 -> unconnected-(U1-GPIO15-Pad20)
- U1 pad 24: AC_IN_3 -> D3
- U1 pad 25: AC_IN_4 -> T1_Pin
- U1 pad 26: D3 -> AC_IN_2
- U1 pad 27: D2 -> AC_IN_1
- U1 pad 28: D1 -> AC_IN_4
- U1 pad 29: T1_Pin -> AC_IN_3
- U1 pad 30: unconnected-(U1-U0RXD/GPIO17-Pad30) -> Net-(J11-Pin_3)
- U1 pad 31: unconnected-(U1-U0TXD/GPIO16-Pad31) -> Net-(J11-Pin_2)
- U1 pad 5: SP2 -> IR_OUT
- U1 pad 6: SP3 -> D1
- U1 pad 9: SP4 -> unconnected-(U1-MTMS/GPIO4/ADC1_CH4-Pad9)
- U4 pad 5: Net-(J9-Pin_1) -> Net-(J9-Pin_2)
- U4 pad 6: Net-(J9-Pin_2) -> Net-(J9-Pin_1)
Routing:
- net +3.3V: track 0.00 -> 144.5 mm, vias 0 -> 5
- net +5V: track 0.00 -> 143.7 mm, vias 0 -> 14
- net Net-(U1-EN/CHIP_PU): track 0.00 -> 56.3 mm, vias 0 -> 3
- net LOAD_F: track 0.00 -> 48.8 mm
- net LOAD_1: track 0.00 -> 47.9 mm
- net AC_IN_4: track 0.00 -> 47.2 mm, vias 0 -> 2
- net Net-(D3-A): track 0.00 -> 47.2 mm, vias 0 -> 1
- net AC_IN_3: track 0.00 -> 46.8 mm, vias 0 -> 3
- net Net-(Q1-G): track 0.00 -> 43.4 mm
- net AC_IN_2: track 0.00 -> 41.9 mm, vias 0 -> 5
- net AC_IN_1: track 0.00 -> 41.9 mm, vias 0 -> 2
- net D1: track 0.00 -> 40.2 mm, vias 0 -> 2
- net LOAD_2: track 0.00 -> 38.9 mm
- net D3: track 0.00 -> 37.1 mm
- net Net-(D2-A): track 0.00 -> 35.5 mm
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Other:
- outline, holes or cut-outs redrawn

Commit message: Major Update
- Removed All 3D related files for now.
- Updated the Schematics and PCB
- Updated the assets
Parts:
- moved J1 7.23 mm to (82.3, 36.8), turned to -90 degrees
Routing:
- net AC_N: track 6.11 -> 86.6 mm, vias 4 -> 3
- net +5V: track 143.7 -> 184.0 mm, vias 14 -> 13
- net AC_L: track 28.0 -> 9.00 mm
- net Net-(J8-CC1): track 30.6 -> 13.4 mm
- net +3.3V: track 144.5 -> 130.2 mm, vias 5 -> 4
- net Net-(U1-GPIO13/USB_D+): track 30.1 -> 17.4 mm, vias 2 -> 0
- net Net-(U1-EN/CHIP_PU): track 56.3 -> 46.3 mm
- net Net-(J8-CC2): track 11.6 -> 21.5 mm
- net Net-(U1-GPIO12/USB_D-): track 26.1 -> 19.7 mm, vias 2 -> 0
- net S3: track 15.7 -> 11.6 mm
- net LOAD_3: track 33.0 -> 36.6 mm, vias 0 -> 1
- net Net-(D11-+): track 14.2 -> 10.5 mm
- net Net-(Q5-E): track 5.26 -> 8.37 mm, vias 0 -> 2
- net Net-(Q1-G): track 43.4 -> 46.5 mm
- net Net-(U4-B_OUT-): track 32.9 -> 35.9 mm, vias 0 -> 2
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Other:
- board text added: "1"
- board text added: "2"
- board text added: "3"
- board text added: "AARAM"
- board text added: "B+"
- board text added: "B-"
- board text added: "By: XICOR22"
- board text added: "D G V DHT22"
- board text added: "DOWN"
- board text added: "F"
- board text added: "IR_OUT G +"
- board text added: "L"
- board text added: "LiPo"
- board text added: "N"
- board text added: "PSU_5V"
- board text added: "PSU_GND"
- board text added: "PSU_IN"
- board text added: "RST"
- board text added: "Switch Input"
- board text added: "TX RX"
- board text added: "V IR_IN G D"
